Commit message: updated with current YOLO progress

File: catkin_ws/src/igvc/urdf/oldRobot.urdf (robot description, URDF)
Before this commit: robot oldRobot, 9 links, 8 joints
Links:
- link base_link: geometry visual box size=0.4878 0.8382 0.0381
Joints:
- joint laser_joint: origin xyz=0 0 .5 rpy=0 0 0 -> xyz=0 0 1.5 rpy=0 .4 0

Commit message: lane-detection code

File: catkin_ws/src/igvc/urdf/oldRobot.urdf (robot description, URDF)
Before this commit: robot oldRobot, 9 links, 8 joints
Links:
- link base_link: geometry collision box size=0.4878 0.8382 0.0381; visual box size=0.4878 0.8382 0.0381
Joints:
- joint laser_joint: origin xyz=0 0 1.5 rpy=0 .4 0 -> xyz=0 0 1.8 rpy=0 0.3 0
